File: KiCAD/Rover V6.kicad_pcb (KiCad board)
At the start: 2 copper layers, 86.4 x 165.1 mm, 36 parts, among them J1 Conn_01x15, J2 Conn_01x15, M1 DC_Motor, M2 DC_Motor, SW1 SW_DPDT_x2, U1 L293D, U2 TP4056_Charger, U3 S-80836CNY-B2-U, U4 74HC123D, U5 MPU-6050

Commit message: Updated Arduino
Parts:
- moved G7 2.16 mm to (89.4, 80.8)
Changed lines of the file:
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@@
-(kicad_pcb (version 20171130) (host pcbnew 5.1.3-ffb9f22~84~ubuntu19.04.1)
+(kicad_pcb (version 20171130) (host pcbnew 5.1.4-e60b266~84~ubuntu19.04.1)
   (general
     (thickness 1.6)
@@
   )
   (module rover:LOGO2 (layer F.Cu)
-    (at 89.408 78.613)
+    (at 89.408 80.772)
     (fp_text reference G7 (at 0 0) (layer F.SilkS) hide
       (effects (font (size 1.524 1.524) (thickness 0.3)))
@@
     (effects (font (size 5 5) (thickness 0.85)))
   )
-  (gr_text "Designed By:\nWilliam E. Gerhard III\nwillig42@vt.edu\nJonathan Z. Kayne\njzkmath@vt.edu" (at 88.392 85.344) (layer F.SilkS)
+  (gr_text "Designed By:\nWilliam E. Gerhard III\nwillig42@vt.edu\nJonathan Z. Kayne\njzkmath@vt.edu" (at 88.9 100.584) (layer F.SilkS)
     (effects (font (size 1 1) (thickness 0.15)))
   )
-  (gr_text "Bumper Car V6\nDesigned: July 31st, 2019\nS/N: HW-LCR03-V6.1A" (at 89.154 73.152) (layer F.SilkS)
+  (gr_text "Bumper Car V6\nDesigned: July 31st, 2019\nS/N: HW-LCR03-V6.1A" (at 89.154 74.676) (layer F.SilkS)
     (effects (font (size 0.8 0.8) (thickness 0.15)))
   )
-  (gr_text ECE@VT (at 89.789 67.564) (layer F.SilkS)
+  (gr_text ECE@VT (at 89.916 69.088) (layer F.SilkS)
     (effects (font (size 5 3) (thickness 0.55)))
   )
